File: bubbler.kicad_pcb (KiCad board)
At the start: 2 copper layers, 30.5 x 29.2 mm, 28 parts, among them J1 Conn_01x04_Pin, U1 LM4041DYM3-1.2, U2 TLV07, U3 INA823DR

Commit message: Settled on design for microblower
Other:
- board text added: "C2 should be 0805 D3 is too tight a fit"
- board text added: "U3 is too wide"
Changed lines of the file:
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@@
+		)
+	)
+	(gr_text "C2 should be 0805\nD3 is too tight a fit"
+		(at 121.92 53.34 0)
+		(layer "Eco1.User")
+		(effects
+			(font
+				(size 1 1)
+				(thickness 0.15)
+			)
+			(justify left bottom)
+		)
+	)
+	(gr_text "U3 is too wide"
+		(at 119.38 86.36 0)
+		(layer "Eco1.User")
+		(effects
+			(font
+				(size 1 1)
+				(thickness 0.15)
+			)
+			(justify left bottom)
 		)
 	)
